File: BedCooler.kicad_sch (KiCad schematic)
At the start: 21 parts, among them J16 Conn_01x05, J20 Conn_01x22_Female, SW1 SW_SPDT, U1 STM32G474RET6, X1 X32258MOB4SI

Commit message: Updated schematic and routed PCB traces
Parts:
- added B1: CR2032-BS-5-1, easyeda2kicad:BAT-TH_CR2032-BS-5-1, symbol easyeda2kicad:CR2032-BS-5-1
Connections:
- net GND: now also B1.2
- net VBAT: now also Module1.76 (VBAT), B1.1
Other:
- sheet H_bridge renamed H bridge (page 2)
- moved on the sheet: C102, C48, C49, C50, C51, C52, C53, C54, C55, C56, C83, C92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

Commit message: Updated schematic and routed PCB
Parts:
- added C103, C104: 100n, Capacitor_SMD:C_0402_1005Metric, symbol Device:C
- added C105: 1uF, Capacitor_SMD:C_0603_1608Metric, symbol Device:C
- added J22: 690-019-298-412, CM5IO:EDAC 690-019-298-412, symbol CM5IO:HDMI_A_1.4
- added J23: Conn_01x02_Pin, Connector_JST:JST_XH_B2B-XH-A_1x02_P2.50mm_Vertical, symbol Connector:Conn_01x02_Pin
- added R65: 10k, Resistor_SMD:R_0603_1608Metric, symbol Device:R
- added R66, R67, R68, R69, R70, R71: 4.7k, Resistor_SMD:R_0603_1608Metric, symbol Device:R
- added R72: 100k, Resistor_SMD:R_0603_1608Metric, symbol Device:R
- added U13: RT9742SNGV, Package_TO_SOT_SMD:TSOT-23_HandSoldering, symbol CM5IO:RT9742SNGV
Connections:
- net +3.3V: now also R68.1, R69.1
- net +5V: now also C103.1, C105.2, J23.1 (Pin_1), U13.1 (IN)
- net GND: now also C103.2, C104.2, C105.1, J22.11 (CKS), J22.17 (GND), J22.2 (D2S), J22.5 (D1S), J22.8 (D0S), J22.SH1 (SH), J22.SH2 (SH), J22.SH3 (SH), J22.SH4 (SH), J23.2 (Pin_2), R72.1, U13.3 (GND); no longer SW1.1 (A)
- net SCL: now also R66.2
- net SCL0: now also R68.2
- net SDA: now also R67.2
- net SDA0: now also R69.2
- net HDMI0_CEC: now reaches Module1.151 (HDMI0_CEC)
- net HDMI0_CEC: now also J22.13 (CEC)
- net HDMI0_HOTPLUG: now reaches Module1.153 (HDMI0_HOTPLUG)
- net HDMI0_HOTPLUG: now also J22.19 (HPD/HEAC-)
- net HDMI0_D2_P: now reaches Module1.170 (HDMI0_TX2_P)
- net HDMI0_D2_P: now also J22.1 (D2+)
- net HDMI0_D2_N: now reaches Module1.172 (HDMI0_TX2_N)
- net HDMI0_D2_N: now also J22.3 (D2-)
- net HDMI0_D1_P: now reaches Module1.176 (HDMI0_TX1_P)
- net HDMI0_D1_P: now also J22.4 (D1+)
- net HDMI0_D1_N: now reaches Module1.178 (HDMI0_TX1_N)
- net HDMI0_D1_N: now also J22.6 (D1-)
- net HDMI0_D0_P: now reaches Module1.182 (HDMI0_TX0_P)
- net HDMI0_D0_P: now also J22.7 (D0+)
- net HDMI0_D0_N: now reaches Module1.184 (HDMI0_TX0_N)
- net HDMI0_D0_N: now also J22.9 (D0-)
- net HDMI0_CK_P: now reaches Module1.188 (HDMI0_CLK_P)
- net HDMI0_CK_P: now also J22.10 (CK+)
- net HDMI0_CK_N: now reaches Module1.190 (HDMI0_CLK_N)
- net HDMI0_CK_N: now also J22.12 (CK-)
- net HDMI0_SDA: now reaches Module1.199 (HDMI0_SDA)
- net HDMI0_SDA: now also J22.16 (SDA), R70.2
- net HDMI0_SCL: now reaches Module1.200 (HDMI0_SCL)
- net HDMI0_SCL: now also J22.15 (SCL), R71.2
- net at Module1.93 (nRPIBOOT): now also R65.2
- net +3.3v 2: now reaches Module1.99 (PMIC_ENABLE)
- new net: R72.2, SW1.1 (A)
- new net +3.3V 2: R65.1, R66.1, R67.1, R70.1, R71.1
- new net HDMI_5v: C104.1, J22.18 (+5V), U13.2 (OUT)
- no-connect marks 0 -> 1
