File: CM5 Ports.kicad_sch (KiCad schematic)
At the start: 19 parts, among them J10 Micro_SD_Card, J17 USB_C_Receptacle_USB2.0_16P, J9 USB3_A, U10 AP22811AW5-7, U12 GL823K-HCY04, U9 AP22811AW5-7

Commit message: Updated schematic and routed PCB
Parts:
- added D6: TPD2EUSB30ADRTR, easyeda2kicad:SOT-9X3-3_L1.0-W0.8-P0.35-LS1.0-BR, symbol easyeda2kicad:TPD2EUSB30ADRTR
- added J21: USB_C_Receptacle_USB2.0_16P, Connector_USB:USB_C_Receptacle_HRO_TYPE-C-31-M-12, symbol Connector:USB_C_Receptacle_USB2.0_16P
- added R42, R43: 5.1k, Resistor_SMD:R_0603_1608Metric, symbol Device:R
- added R62, R63: 22, Resistor_SMD:R_0603_1608Metric, symbol Device:R
- added U11: AP22811AW5-7, easyeda2kicad:SOT-25-5_L3.0-W1.6-P0.95-LS2.8-BL, symbol easyeda2kicad:AP22811AW5-7
- R46, R47: value 5.1k -> 56k
Connections:
- net +5V: now also R46.2, R47.2, U11.5 (IN)
- net GND: now also D6.3 (GND), J21.A1 (GND), J21.A12 (GND), J21.B1 (GND), J21.B12 (GND), J21.S1 (SHIELD), R42.2, R43.2, U11.2 (GND); no longer R46.2, R47.2
- new net: J21.A4 (VBUS), J21.A9 (VBUS), J21.B4 (VBUS), J21.B9 (VBUS), U11.1 (OUT)
- new net: J21.A5 (CC1), R42.1
- new net: J21.A6 (D+), J21.B6 (D+), R63.1
- new net: J21.A7 (D-), J21.B7 (D-), R62.1
- new net: J21.B5 (CC2), R43.1
- new net PC8: U11.4 (EN/~{EN})
- new net StmUSb+: D6.1 (D+), R63.2
- new net StmUSb-: D6.2 (D-), R62.2
